Commit message: refactor(origincar_description): 重构 URDF 为参数化 xacro，新增 STL 网格版模型

File: src/origincar/origincar_description/urdf/origincar.xacro (robot description, xacro)
@@ -4,133 +4,109 @@
   <xacro:property name="Track" value="0.1682"/>
   <xacro:property name="WheelBase" value="0.189"/>
-  <xacro:property name="WheelLen" value="0.025"/>
+  <xacro:property name="WheelRadius" value="0.03"/>
+  <xacro:property name="BaseBoxLength" value="0.276"/>
+  <xacro:property name="BaseBoxWidth" value="0.164"/>
+  <xacro:property name="BaseBoxHeight" value="0.08"/>
+  <xacro:macro name="wheel" params="prefix side_x side_y">
+    <link name="${prefix}_Link">
+      <visual>
+        <origin xyz="0 0 0" rpy="${side_y * (-PI / 2)} 0 0"/>
+        <geometry>
+          <cylinder radius="${WheelRadius}" length="0.025"/>
+        </geometry>
+        <material name="">
+          <color rgba="0.21176470588235294 0.16470588235294117 0.16470588235294117 1.0"/>
+        </material>
+      </visual>
+    </link>
+    <joint name="${prefix}_joint" type="continuous">
+      <parent link="base_link"/>
+      <child link="${prefix}_Link"/>
+      <origin xyz="${side_x * Track / 2} ${side_y * WheelBase / 2} ${WheelRadius}" rpy="0 0 0"/>
+      <axis xyz="0 ${side_y} 0"/>
+    </joint>
+  </xacro:macro>
+  <link name="base_footprint"/>
+  <joint name="base_footprint_joint" type="fixed">
+    <parent link="base_footprint"/>
+    <child link="base_link"/>
+    <origin xyz="0 0 ${WheelRadius}" rpy="0 0 0"/>
+  </joint>
   <link name="base_link">
     <visual>
       <geometry>
-        <box size="0.276 ${WheelBase-WheelLen} 0.08"/>
+        <box size="${BaseBoxLength} ${BaseBoxWidth} ${BaseBoxHeight}"/>
       </geometry>
-      <origin xyz="0 0 ${0.08/2+0.03}" rpy="0 0 0"/>
-      <material name="rgba(102,10,10,1)">
-        <color rgba="${102/255} ${10/255} ${10/255} 1" />
+      <origin xyz="0 0 ${BaseBoxHeight / 2 + WheelRadius}" rpy="0 0 0"/>
+      <material name="rgb(54, 42, 42)">
+        <color rgba="0.21176470588235294 0.16470588235294117 0.16470588235294117 1.0"/>
       </material>
     </visual>
   </link>
+  <link name="gyro_link"/>
+  <joint name="gyro_joint" type="fixed">
+    <parent link="base_link"/>
+    <child link="gyro_link"/>
+    <origin xyz="0 0 0" rpy="0 0 0"/>
+  </joint>
   <link name="board_link">
     <visual>
       <geometry>
-        <box size="0.200 ${WheelBase-WheelLen} ${0.150-0.08}"/>
+        <box size="0.200 ${BaseBoxWidth} 0.07"/>
       </geometry>
-      <origin xyz="0 0 ${(0.150-0.08)/2}" rpy="0 0 0"/>
+      <origin xyz="0 0 0.035" rpy="0 0 0"/>
       <material name="rgba(246,152,152,1)">
-        <color rgba="${246/255} ${152/255} ${152/255} 1" />
+        <color rgba="0.9647058823529412 0.596078431372549 0.596078431372549 1"/>
       </material>
     </visual>
   </link>
-  <link name="camera" >
+  <link name="camera">
     <visual>
       <geometry>
         <box size="0.015 0.045 0.03"/>
       </geometry>
-      <origin xyz="0 0 ${(0.03)/2}" rpy="0 0 0"/>
+      <origin xyz="0 0 0.015" rpy="0 0 0"/>
       <material name="rgba(93,78,78,1)">
-        <color rgba="${93/255} ${78/255} ${78/255} 1" />
+        <color rgba="0.36470588235294116 0.3058823529411765 0.3058823529411765 1"/>
       </material>
     </visual>
   </link>
   <joint name="camera_joint" type="fixed">
-    <parent link="base_link" />
-    <child link="camera" />
-    <origin xyz="${(0.276-0.015)/2-0.01} 0 ${0.08+0.03}" rpy="0 0 0" />
+    <parent link="base_link"/>
+    <child link="camera"/>
+    <origin xyz="${(BaseBoxLength - 0.015) / 2 - 0.01} 0 ${WheelRadius + BaseBoxHeight}" rpy="0 0 0"/>
   </joint>
   <joint name="board_joint" type="fixed">
-    <parent link="base_link" />
-    <child link="board_link" />
-    <origin xyz="${-(0.276-0.2)/2} 0 ${0.08+0.03}" rpy="0 0 0" />
-    <axis xyz="0 1 0" />
+    <parent link="base_link"/>
+    <child link="board_link"/>
+    <origin xyz="${-(BaseBoxLength - 0.200) / 2} 0 ${WheelRadius + BaseBoxHeight}" rpy="0 0 0"/>
+    <axis xyz="0 1 0"/>
   </joint>
-  <link name="down_left_Link">
+  <xacro:wheel prefix="down_left"  side_x="-1" side_y="1"/>
+  <xacro:wheel prefix="down_right" side_x="-1" side_y="-1"/>
+  <xacro:wheel prefix="up_left"    side_x="1"  side_y="1"/>
+  <xacro:wheel prefix="up_right"   side_x="1"  side_y="-1"/>
+  <link name="laser">
     <visual>
-      <origin xyz="0 ${-WheelLen/2+0.025/2} 0" rpy="${-PI/2} 0 0" />
+      <origin xyz="0 0 0.015" rpy="0 0 0"/>
       <geometry>
-        <cylinder radius="0.03" length="0.025" />
+        <cylinder length="0.03" radius="0.025"/>
       </geometry>
-      <material name="">
-        <color rgba="0.7450980392156863 0.12941176470588237 0.12941176470588237 1" />
+      <material name="dark_brown">
+        <color rgba="0.21176470588235294 0.16470588235294117 0.16470588235294117 1.0"/>
       </material>
     </visual>
-  </link>
-  <joint name="down_left_joint" type="continuous">
-    <parent link="base_link" />
-    <child link="down_left_Link" />
-    <origin xyz="${-Track/2} ${WheelBase/2} ${0.03}" rpy="0 0 0" />
-    <axis xyz="0 1 0" />
-  </joint>
-  <link name="down_right_Link">
     <visual>
-      <origin xyz="0 ${WheelLen/2-0.025/2} 0" rpy="${PI/2} 0 0" />
+      <origin xyz="0 0 0.035" rpy="0 0 0"/>
       <geometry>
-        <cylinder radius="0.03" length="0.025"/>
+        <cylinder length="0.01" radius="0.020"/>
       </geometry>
-      <material name="">
-        <color rgba="0.7450980392156863 0.12941176470588237 0.12941176470588237 1" />
-      </material>
-    </visual>
-  </link>
-  <joint name="down_right_joint" type="continuous">
-    <parent link="base_link" />
-    <child link="down_right_Link" />
-    <origin xyz="${-Track/2} ${-WheelBase/2} ${0.03}" rpy="0 0 0" />
-    <axis xyz="0 -1 0" />
-  </joint>
-  <link name="up_left_Link">
-    <visual>
-      <origin xyz="0 ${-WheelLen/2+0.025/2} 0" rpy="${-PI/2} 0 0" />
-      <geometry>
-        <cylinder radius="0.03" length="0.025"/>
-      </geometry>
-      <material name="">
-        <color rgba="0.7450980392156863 0.12941176470588237 0.12941176470588237 1" />
-      </material>
-    </visual>
-  </link>
-  <joint name="up_left_joint" type="continuous">
-    <parent link="base_link" />
-    <child  link="up_left_Link" />
-    <origin xyz="${Track/2} ${WheelBase/2} ${0.03}" rpy="0 0 0" />
-    <axis xyz="0 1 0" />
-  </joint>
-  <link name="up_right_Link">
-    <visual>
-      <origin xyz="0 ${WheelLen/2-0.025/2} 0" rpy="${PI/2} 0 0" />
-      <geometry>
-        <cylinder radius="0.03" length="0.025"/>
-      </geometry>
-      <material name="">
-        <color rgba="0.7450980392156863 0.12941176470588237 0.12941176470588237 1" />
-      </material>
-    </visual>
-  </link>
-  <joint name="up_right_joint" type="continuous">
-    <parent link="base_link" />
-    <child link="up_right_Link" />
-    <origin xyz="${Track/2} ${-WheelBase/2} ${0.03}" rpy="0 0 0" />
-    <axis  xyz="0 -1 0" />
-  </joint>
-  <!-- 激光雷达模型 -->
-  <link name="laser_link">
-    <visual>
-      <origin xyz="0 0 0" rpy="0 0 0" />
-      <geometry>
-        <cylinder radius="0.04" length="0.05"/>
-      </geometry>
-      <material name="">
-        <color rgba="0.2 0.2 0.2 1" />
-      </material>
+      <material name="dark_brown"/>
     </visual>
   </link>
   <joint name="laser_joint" type="fixed">
-    <parent link="base_link" />
-    <child link="laser_link" />
-    <origin xyz="0.15 0 0.12" rpy="0 0 0" />
+    <parent link="board_link"/>
+    <child link="laser"/>
+    <origin xyz="0.073 0 0.07" rpy="0 0 0"/>
   </joint>
 </robot>

Commit message: feat(origincar_description): 重构URDF为阿克曼转向模型
- 将差速驱动模型改为阿克曼转向模型
- 前轮添加转向关节(revolute)和驱动关节(continuous)
- 后轮仅保留驱动关节(continuous)
- 转向限位±0.55rad(31.5°)
- 左侧轮子绕Z轴旋转180°对称
- STL版材质统一为dark_grey

File: src/origincar/origincar_description/urdf/origincar.xacro (robot description, xacro)
@@ -1,30 +1,77 @@
 <?xml version="1.0" encoding="utf-8"?>
 <robot name="mycar" xmlns:xacro="http://wiki.ros.org/xacro">
+  <!-- 基础参数 -->
   <xacro:property name="PI" value="3.1415926"/>
   <xacro:property name="Track" value="0.1682"/>
   <xacro:property name="WheelBase" value="0.189"/>
   <xacro:property name="WheelRadius" value="0.03"/>
+  <xacro:property name="WheelWidth" value="0.025"/>
   <xacro:property name="BaseBoxLength" value="0.276"/>
   <xacro:property name="BaseBoxWidth" value="0.164"/>
   <xacro:property name="BaseBoxHeight" value="0.08"/>
-  <xacro:macro name="wheel" params="prefix side_x side_y">
-    <link name="${prefix}_Link">
+  <xacro:property name="SteerLinkLength" value="0.02"/>
+  <!-- 前轮转向宏 -->
+  <xacro:macro name="front_wheel" params="prefix side_y">
+    <!-- 转向关节连接的link -->
+    <link name="${prefix}_steer_link">
+      <visual>
+        <origin xyz="0 0 0" rpy="0 0 0"/>
+        <geometry>
+          <cylinder radius="0.008" length="${SteerLinkLength}"/>
+        </geometry>
+        <material name="steer_mat">
+          <color rgba="0.5 0.5 0.5 1.0"/>
+        </material>
+      </visual>
+    </link>
+    <!-- 转向关节（绕Z轴旋转） -->
+    <joint name="${prefix}_steer_joint" type="revolute">
+      <parent link="base_link"/>
+      <child link="${prefix}_steer_link"/>
+      <origin xyz="${WheelBase / 2} ${side_y * Track / 2} ${WheelRadius}" rpy="0 0 0"/>
+      <axis xyz="0 0 1"/>
+      <limit lower="-0.55" upper="0.55" effort="100" velocity="10"/>
+    </joint>
+    <!-- 驱动轮link -->
+    <link name="${prefix}_wheel_link">
       <visual>
         <origin xyz="0 0 0" rpy="${side_y * (-PI / 2)} 0 0"/>
         <geometry>
-          <cylinder radius="${WheelRadius}" length="0.025"/>
+          <cylinder radius="${WheelRadius}" length="${WheelWidth}"/>
         </geometry>
-        <material name="">
+        <material name="wheel_mat">
           <color rgba="0.21176470588235294 0.16470588235294117 0.16470588235294117 1.0"/>
         </material>
       </visual>
     </link>
-    <joint name="${prefix}_joint" type="continuous">
-      <parent link="base_link"/>
-      <child link="${prefix}_Link"/>
-      <origin xyz="${side_x * Track / 2} ${side_y * WheelBase / 2} ${WheelRadius}" rpy="0 0 0"/>
+    <!-- 驱动关节（绕Y轴旋转） -->
+    <joint name="${prefix}_wheel_joint" type="continuous">
+      <parent link="${prefix}_steer_link"/>
+      <child link="${prefix}_wheel_link"/>
+      <origin xyz="0 0 0" rpy="0 0 0"/>
       <axis xyz="0 ${side_y} 0"/>
     </joint>
   </xacro:macro>
+  <!-- 后轮驱动宏 -->
+  <xacro:macro name="rear_wheel" params="prefix side_y">
+    <link name="${prefix}_wheel_link">
+      <visual>
+        <origin xyz="0 0 0" rpy="${side_y * (-PI / 2)} 0 0"/>
+        <geometry>
+          <cylinder radius="${WheelRadius}" length="${WheelWidth}"/>
+        </geometry>
+        <material name="wheel_mat">
+          <color rgba="0.21176470588235294 0.16470588235294117 0.16470588235294117 1.0"/>
+        </material>
+      </visual>
+    </link>
+    <joint name="${prefix}_wheel_joint" type="continuous">
+      <parent link="base_link"/>
+      <child link="${prefix}_wheel_link"/>
+      <origin xyz="${-WheelBase / 2} ${side_y * Track / 2} ${WheelRadius}" rpy="0 0 0"/>
+      <axis xyz="0 ${side_y} 0"/>
+    </joint>
+  </xacro:macro>
+  <!-- base_footprint -->
   <link name="base_footprint"/>
   <joint name="base_footprint_joint" type="fixed">
@@ -33,4 +80,5 @@
     <origin xyz="0 0 ${WheelRadius}" rpy="0 0 0"/>
   </joint>
+  <!-- 车体 -->
   <link name="base_link">
     <visual>
@@ -44,4 +92,5 @@
     </visual>
   </link>
+  <!-- IMU link -->
   <link name="gyro_link"/>
   <joint name="gyro_joint" type="fixed">
@@ -50,4 +99,5 @@
     <origin xyz="0 0 0" rpy="0 0 0"/>
   </joint>
+  <!-- 电路板 -->
   <link name="board_link">
     <visual>
@@ -61,4 +111,10 @@
     </visual>
   </link>
+  <joint name="board_joint" type="fixed">
+    <parent link="base_link"/>
+    <child link="board_link"/>
+    <origin xyz="${-(BaseBoxLength - 0.200) / 2} 0 ${WheelRadius + BaseBoxHeight}" rpy="0 0 0"/>
+  </joint>
+  <!-- 摄像头 -->
   <link name="camera">
     <visual>
@@ -77,14 +133,11 @@
     <origin xyz="${(BaseBoxLength - 0.015) / 2 - 0.01} 0 ${WheelRadius + BaseBoxHeight}" rpy="0 0 0"/>
   </joint>
-  <joint name="board_joint" type="fixed">
-    <parent link="base_link"/>
-    <child link="board_link"/>
-    <origin xyz="${-(BaseBoxLength - 0.200) / 2} 0 ${WheelRadius + BaseBoxHeight}" rpy="0 0 0"/>
-    <axis xyz="0 1 0"/>
-  </joint>
-  <xacro:wheel prefix="down_left"  side_x="-1" side_y="1"/>
-  <xacro:wheel prefix="down_right" side_x="-1" side_y="-1"/>
-  <xacro:wheel prefix="up_left"    side_x="1"  side_y="1"/>
-  <xacro:wheel prefix="up_right"   side_x="1"  side_y="-1"/>
+  <!-- 前轮（转向+驱动） -->
+  <xacro:front_wheel prefix="front_left"  side_y="1"/>
+  <xacro:front_wheel prefix="front_right" side_y="-1"/>
+  <!-- 后轮（仅驱动） -->
+  <xacro:rear_wheel prefix="rear_left"  side_y="1"/>
+  <xacro:rear_wheel prefix="rear_right" side_y="-1"/>
+  <!-- 激光雷达 -->
   <link name="laser">
     <visual>

File: src/origincar/origincar_description/urdf/origincar_stl.xacro (robot description, xacro)
@@ -1,4 +1,6 @@
 <?xml version="1.0" encoding="utf-8"?>
 <robot name="mycar" xmlns:xacro="http://wiki.ros.org/xacro">
+  <!-- 基础参数 -->
+  <xacro:property name="PI" value="3.1415926"/>
   <xacro:property name="FrontWheelX" value="0.06"/>
   <xacro:property name="RearWheelX" value="0.0841"/>
@@ -6,14 +8,56 @@
   <xacro:property name="WheelZ" value="0.025"/>
   <xacro:property name="base_link_Z" value="0.01"/>
-  <xacro:macro name="wheel" params="prefix x y z axis_sign">
+  <xacro:property name="SteerLinkLength" value="0.002"/>
+  <xacro:property name="SteerPivotX" value="0.06"/>
+  <material name="dark_grey">
+    <color rgba="0.2 0.2 0.2 1.0"/>
+  </material>
+  <!-- 前轮转向宏 -->
+  <xacro:macro name="front_wheel" params="prefix y axis_sign yaw steer_link_y steer_joint_y joint_y">
+    <!-- 转向关节连接的link -->
+    <link name="${prefix}_steer_link">
+      <visual>
+        <origin xyz="0 ${steer_link_y} 0" rpy="${PI/2} 0 0"/>
+        <geometry>
+          <cylinder radius="0.0018" length="${SteerLinkLength}"/>
+        </geometry>
+        <material name="dark_grey"/>
+      </visual>
+    </link>
+    <!-- 转向关节（绕Z轴旋转） -->
+    <joint name="${prefix}_steer_joint" type="revolute">
+      <parent link="base_link"/>
+      <child link="${prefix}_steer_link"/>
+      <origin xyz="${SteerPivotX} ${steer_joint_y} ${WheelZ}" rpy="0 0 0"/>
+      <axis xyz="0 0 1"/>
+      <limit lower="-0.55" upper="0.55" effort="100" velocity="10"/>
+    </joint>
+    <!-- 驱动轮link -->
     <link name="${prefix}_Link">
       <visual>
-        <origin xyz="0 0 0" rpy="0 0 0"/>
+        <origin xyz="0 0 0" rpy="0 0 ${yaw}"/>
         <geometry>
           <mesh filename="package://origincar_description/meshes/${prefix}_Link.STL"/>
         </geometry>
-        <material name="">
-          <color rgba="0.21176470588235294 0.16470588235294117 0.16470588235294117 1.0"/>
-        </material>
+        <material name="dark_grey"/>
+      </visual>
+    </link>
+    <!-- 驱动关节（绕Y轴旋转） -->
+    <joint name="${prefix}_joint" type="continuous">
+      <parent link="${prefix}_steer_link"/>
+      <child link="${prefix}_Link"/>
+      <origin xyz="0 ${joint_y} 0" rpy="0 0 0"/>
+      <axis xyz="0 ${axis_sign} 0"/>
+    </joint>
+  </xacro:macro>
+  <!-- 后轮驱动宏 -->
+  <xacro:macro name="rear_wheel" params="prefix y axis_sign yaw">
+    <link name="${prefix}_Link">
+      <visual>
+        <origin xyz="0 0 0" rpy="0 0 ${yaw}"/>
+        <geometry>
+          <mesh filename="package://origincar_description/meshes/${prefix}_Link.STL"/>
+        </geometry>
+        <material name="dark_grey"/>
       </visual>
     </link>
@@ -21,8 +65,9 @@
       <parent link="base_link"/>
       <child link="${prefix}_Link"/>
-      <origin xyz="${x} ${y} ${z}" rpy="0 0 0"/>
+      <origin xyz="${-RearWheelX} ${y} ${WheelZ}" rpy="0 0 0"/>
       <axis xyz="0 ${axis_sign} 0"/>
     </joint>
   </xacro:macro>
+  <!-- base_footprint -->
   <link name="base_footprint"/>
   <joint name="base_footprint_joint" type="fixed">
@@ -31,4 +76,5 @@
     <origin xyz="0 0 ${base_link_Z}" rpy="0 0 0"/>
   </joint>
+  <!-- 车体 -->
   <link name="base_link">
     <visual>
@@ -37,9 +83,8 @@
         <mesh filename="package://origincar_description/meshes/base_link.STL"/>
       </geometry>
-      <material name="rgb(54, 42, 42)">
-        <color rgba="0.21176470588235294 0.16470588235294117 0.16470588235294117 1.0"/>
-      </material>
+      <material name="dark_grey"/>
     </visual>
   </link>
+  <!-- IMU link -->
   <link name="gyro_link"/>
   <joint name="gyro_joint" type="fixed">
@@ -48,8 +93,11 @@
     <origin xyz="0 0 0" rpy="0 0 0"/>
   </joint>
-  <xacro:wheel prefix="down_left"  x="${-RearWheelX}" y="${WheelY}"  z="${WheelZ}" axis_sign="1"/>
-  <xacro:wheel prefix="down_right" x="${-RearWheelX}" y="${-WheelY}" z="${WheelZ}" axis_sign="-1"/>
-  <xacro:wheel prefix="up_left"    x="${FrontWheelX}" y="${WheelY}"  z="${WheelZ}" axis_sign="1"/>
-  <xacro:wheel prefix="up_right"   x="${FrontWheelX}" y="${-WheelY}" z="${WheelZ}" axis_sign="-1"/>
+  <!-- 前轮（转向+驱动） -->
+  <xacro:front_wheel prefix="up_left"  y="${WheelY}"  axis_sign="1"  yaw="${PI}" steer_link_y="0.033" steer_joint_y="0.05" joint_y="0.03"/>
+  <xacro:front_wheel prefix="up_right" y="${-WheelY}" axis_sign="-1" yaw="0" steer_link_y="-0.033" steer_joint_y="-0.05" joint_y="-0.03"/>
+  <!-- 后轮（仅驱动） -->
+  <xacro:rear_wheel prefix="down_left"  y="${WheelY}"  axis_sign="1"  yaw="${PI}"/>
+  <xacro:rear_wheel prefix="down_right" y="${-WheelY}" axis_sign="-1" yaw="0"/>
+  <!-- 激光雷达 -->
   <link name="laser">
     <visual>
@@ -58,7 +106,5 @@
         <mesh filename="package://origincar_description/meshes/lslidar_N10.stl"/>
       </geometry>
-      <material name="dark_brown">
-        <color rgba="0.21176470588235294 0.16470588235294117 0.16470588235294117 1.0"/>
-      </material>
+      <material name="dark_grey"/>
     </visual>
   </link>
