Commit message: feat(origincar_description): 添加镭神N10雷达STL模型并替换laser link占位圆柱体

File: src/origincar/origincar_description/urdf/origincar_stl.xacro (robot description, xacro)
@@ -56,14 +56,5 @@
       <origin xyz="0 0 0" rpy="0 0 0"/>
       <geometry>
-        <cylinder length="0.025" radius="0.025"/>
-      </geometry>
-      <material name="dark_brown">
-        <color rgba="0.21176470588235294 0.16470588235294117 0.16470588235294117 1.0"/>
-      </material>
-    </visual>
-    <visual>
-      <origin xyz="0 0 0.015" rpy="0 0 0"/>
-      <geometry>
-        <cylinder length="0.01" radius="0.020"/>
+        <mesh filename="package://origincar_description/meshes/lslidar_N10.stl"/>
       </geometry>
       <material name="dark_brown">
@@ -75,5 +66,5 @@
     <parent link="base_link"/>
     <child link="laser"/>
-    <origin xyz="0.025 0 0.135" rpy="0 0 0"/>
+    <origin xyz="0.02 0.02 0.145" rpy="0 0 4.755"/>
   </joint>
 </robot>

Commit message: feat(description): 优化机器人模型和激光雷达姿态
- 新增 base_link1.STL 和 top_link.stl 模型文件
- 调整激光雷达 roll 角度至 0.03 弧度

File: src/origincar/origincar_description/urdf/origincar_stl.xacro (robot description, xacro)
@@ -102,5 +102,5 @@
   <link name="laser">
     <visual>
-      <origin xyz="0 0 0" rpy="0 0 0"/>
+      <origin xyz="0 0 0" rpy="0.03 0 0"/>
       <geometry>
         <mesh filename="package://origincar_description/meshes/lslidar_N10.stl"/>

Commit message: perf: 优化STL模型

File: src/origincar/origincar_description/urdf/origincar_stl.xacro (robot description, xacro)
@@ -7,9 +7,15 @@
   <xacro:property name="WheelY" value="0.08"/>
   <xacro:property name="WheelZ" value="0.025"/>
-  <xacro:property name="base_link_Z" value="0.01"/>
+  <xacro:property name="base_link_Z" value="0.02"/>
   <xacro:property name="SteerLinkLength" value="0.002"/>
   <xacro:property name="SteerPivotX" value="0.06"/>
+  <material name="black">
+    <color rgba="0.1 0.1 0.1 1.0"/>
+  </material>
   <material name="dark_grey">
     <color rgba="0.2 0.2 0.2 1.0"/>
+  </material>
+  <material name="pink">
+    <color rgba="1.0 0.75 0.8 1.0"/>
   </material>
   <!-- 前轮转向宏 -->
@@ -38,7 +44,7 @@
         <origin xyz="0 0 0" rpy="0 0 ${yaw}"/>
         <geometry>
-          <mesh filename="package://origincar_description/meshes/${prefix}_Link.STL"/>
+          <mesh filename="package://origincar_description/meshes/origincar_wheel.STL"/>
         </geometry>
-        <material name="dark_grey"/>
+        <material name="black"/>
       </visual>
     </link>
@@ -57,7 +63,7 @@
         <origin xyz="0 0 0" rpy="0 0 ${yaw}"/>
         <geometry>
-          <mesh filename="package://origincar_description/meshes/${prefix}_Link.STL"/>
+          <mesh filename="package://origincar_description/meshes/origincar_wheel.STL"/>
         </geometry>
-        <material name="dark_grey"/>
+        <material name="black"/>
       </visual>
     </link>
@@ -71,5 +77,5 @@
   <!-- base_footprint -->
   <link name="base_footprint"/>
-  <joint name="base_footprint_joint" type="fixed">
+  <joint name="base_link_joint" type="fixed">
     <parent link="base_footprint"/>
     <child link="base_link"/>
@@ -79,11 +85,26 @@
   <link name="base_link">
     <visual>
-      <origin xyz="0 0 ${base_link_Z}" rpy="0 0 0"/>
+      <origin xyz="0.0125 0 0.04" rpy="0 0 0"/>
       <geometry>
-        <mesh filename="package://origincar_description/meshes/base_link.STL"/>
+        <mesh filename="package://origincar_description/meshes/origincar_base.STL"/>
       </geometry>
-      <material name="dark_grey"/>
+      <material name="black"/>
     </visual>
   </link>
+  <!-- 车顶 -->
+  <link name="top_link">
+    <visual>
+      <origin xyz="-0.018 0 0" rpy="0 0 0"/>
+      <geometry>
+        <mesh filename="package://origincar_description/meshes/origincar_top.stl"/>
+      </geometry>
+      <material name="pink"/>
+    </visual>
+  </link>
+  <joint name="top_link_joint" type="fixed">
+    <parent link="base_link"/>
+    <child link="top_link"/>
+    <origin xyz="0 0 0.0968" rpy="0 0 0"/>
+  </joint>
   <!-- IMU link -->
   <link name="gyro_link"/>
@@ -102,5 +123,5 @@
   <link name="laser">
     <visual>
-      <origin xyz="0 0 0" rpy="0.03 0 0"/>
+      <origin xyz="0.02 0 0" rpy="0 0 0"/>
       <geometry>
         <mesh filename="package://origincar_description/meshes/lslidar_N10.stl"/>
@@ -110,7 +131,22 @@
   </link>
   <joint name="laser_joint" type="fixed">
+    <parent link="top_link"/>
+    <child link="laser"/>
+    <origin xyz="-0.01 0 0.048" rpy="0 0 0"/>
+  </joint>
+<!-- 摄像头 -->
+  <link name="camera_link">
+    <visual>
+      <origin xyz="0 0 0" rpy="0 0 0"/>
+      <geometry>
+        <mesh filename="package://origincar_description/meshes/origincar_camera.stl"/>
+      </geometry>
+      <material name="dark_grey"/>
+    </visual>
+  </link>
+  <joint name="camera_joint" type="fixed">
     <parent link="base_link"/>
-    <child link="laser"/>
-    <origin xyz="0.02 0.02 0.145" rpy="0 0 4.755"/>
+    <child link="camera_link"/>
+    <origin xyz="0.09 0 0.09" rpy="0 0 0"/>
   </joint>
 </robot>
